Commit message: 2023-05-06 22:13:44
 lgv_description/urdf/lgv_description.urdf.xacro | 4 ++--
 lgv_navigation/maps/map.yaml                    | 3 +--
 lgv_navigation/maps/sim_map.yaml                | 4 ++--
 lgv_simulation/launch/simulation.launch         | 9 ++++++++-
 4 files changed, 13 insertions(+), 7 deletions(-)

File: lgv_description/urdf/lgv_description.urdf.xacro (robot description, xacro)
@@ -2,8 +2,8 @@
 <robot name="lgv_description" xmlns:xacro="http://ros.org/wiki/xacro">
   <xacro:include filename="$(find lgv_description)/urdf/lgv_description.gazebo.xacro" />
-  <link name="base_footprint" />
+  <link name="dummy" />
   <joint name="base_joint" type="fixed">
     <origin xyz="0 0 0" rpy="0 0 0" />
-    <parent link="base_footprint" />
+    <parent link="dummy" />
     <child link="base_link" />
   </joint>
